Commit message: Fix Tibia Joint Orient

File: src/hexapod_description/urdf/Hexapod.urdf (robot description, URDF)
Before this commit: robot Hexapod, 26 links, 25 joints
Joints:
- joint L_back_femur_jnt: axis 0 0 1.0 -> 1.0 0 0
- joint L_back_tibia_jnt: axis 0 0 -1.0 -> -1.0 0 0
- joint L_front_femur_jnt: axis 0 0 1.0 -> 1.0 0 0
- joint L_front_tibia_jnt: axis 0 0 -1.0 -> -1.0 0 0
- joint L_mid_femur_jnt: axis 0 0 1.0 -> 1.0 0 0
- joint L_mid_tibia_jnt: axis 0 0 -1.0 -> -1.0 0 0
- joint R_back_coxa_jnt: axis 0 0 -1.0 -> 0 0 1.0
- joint R_back_femur_jnt: axis 0 0 1.0 -> 1.0 0 0
- joint R_back_tibia_jnt: axis 0 0 -1.0 -> -1.0 0 0
- joint R_front_coxa_jnt: axis 0 0 -1.0 -> 0 0 1.0
- joint R_front_femur_jnt: axis 0 0 1.0 -> 1.0 0 0
- joint R_front_tibia_jnt: axis 0 0 -1.0 -> -1.0 0 0
- joint R_mid_coxa_jnt: axis 0 0 -1.0 -> 0 0 1.0
- joint R_mid_femur_jnt: axis 0 0 1.0 -> 1.0 0 0
- joint R_mid_tibia_jnt: axis 0 0 -1.0 -> -1.0 0 0

Commit message: hexapod urdf and MoveIt package update

File: src/hexapod_description/urdf/Hexapod.urdf (robot description, URDF)
Before this commit: robot Hexapod, 26 links, 25 joints
Links:
- removed link L_back_coxa_jnt
- removed link L_back_femur_jnt
- removed link L_back_foot_jnt
- removed link L_back_tibia_jnt
- removed link L_front_coxa_jnt
- removed link L_front_femur_jnt
- removed link L_front_foot_jnt
- removed link L_front_tibia_jnt
- removed link L_mid_coxa_jnt
- removed link L_mid_femur_jnt
- removed link L_mid_foot_jnt
- removed link L_mid_tibia_jnt
- removed link R_back_coxa_jnt
- removed link R_back_femur_jnt
- removed link R_back_foot_jnt
- removed link R_back_tibia_jnt
- removed link R_front_coxa_jnt
- removed link R_front_femur_jnt
- removed link R_front_foot_jnt
- removed link R_front_tibia_jnt
- removed link R_mid_coxa_jnt
- removed link R_mid_femur_jnt
- removed link R_mid_foot_jnt
- removed link R_mid_tibia_jnt
- removed link body_jnt
- removed link root_jnt
- added link L_back_coxa_link, mass 0.1; collision box size=0.05 0.05964 0.06371; visual mesh filename=package://hexapod_description/meshes/dae/L_coxa_shape.dae scale=1.0 1.0 1.0
- added link L_back_ee_link
- added link L_back_femur_link, mass 0.1; collision box size=0.10497 0.0249 0.002; visual mesh filename=package://hexapod_description/meshes/dae/L_femur_shape.dae scale=1.0 1.0 1.0
- added link L_back_foot_link, mass 0.001
- added link L_back_tibia_link, mass 0.2; collision mesh filename=package://hexapod_description/meshes/dae/L_tibia_shape.003.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 scale=1.0 1.0 1.0; visual mesh filename=package://hexapod_description/meshes/dae/L_tibia_shape.dae scale=1.0 1.0 1.0
- added link L_front_coxa_link, mass 0.1; collision box size=0.05 0.05964 0.06371; visual mesh filename=package://hexapod_description/meshes/dae/L_coxa_shape.dae scale=1.0 1.0 1.0
- added link L_front_ee_link
- added link L_front_femur_link, mass 0.1; collision box size=0.10497 0.0249 0.002; visual mesh filename=package://hexapod_description/meshes/dae/L_femur_shape.dae scale=1.0 1.0 1.0
- added link L_front_foot_link, mass 0.001
- added link L_front_tibia_link, mass 0.2; collision mesh filename=package://hexapod_description/meshes/dae/L_tibia_shape.001.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 scale=1.0 1.0 1.0; visual mesh filename=package://hexapod_description/meshes/dae/L_tibia_shape.dae scale=1.0 1.0 1.0
- added link L_mid_coxa_link, mass 0.1; collision box size=0.05 0.05964 0.06371; visual mesh filename=package://hexapod_description/meshes/dae/L_coxa_shape.dae scale=1.0 1.0 1.0
- added link L_mid_ee_link
- added link L_mid_femur_link, mass 0.1; collision box size=0.10497 0.0249 0.002; visual mesh filename=package://hexapod_description/meshes/dae/L_femur_shape.dae scale=1.0 1.0 1.0
- added link L_mid_foot_link, mass 0.001
- added link L_mid_tibia_link, mass 0.2; collision mesh filename=package://hexapod_description/meshes/dae/L_tibia_shape.002.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 scale=1.0 1.0 1.0; visual mesh filename=package://hexapod_description/meshes/dae/L_tibia_shape.dae scale=1.0 1.0 1.0
- added link R_back_coxa_link, mass 0.1; collision box size=0.05 0.05964 0.06371; visual mesh filename=package://hexapod_description/meshes/dae/R_coxa_shape.dae scale=1.0 1.0 1.0
- added link R_back_ee_link
- added link R_back_femur_link, mass 0.1; collision box size=0.10497 0.0249 0.002; visual mesh filename=package://hexapod_description/meshes/dae/R_femur_shape.dae scale=1.0 1.0 1.0
- added link R_back_foot_link, mass 0.001
- added link R_back_tibia_link, mass 0.2; collision mesh filename=package://hexapod_description/meshes/dae/R_tibia_shape.002.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 scale=1.0 1.0 1.0; visual mesh filename=package://hexapod_description/meshes/dae/R_tibia_shape.dae scale=1.0 1.0 1.0
- added link R_front_coxa_link, mass 0.1; collision box size=0.05 0.05964 0.06371; visual mesh filename=package://hexapod_description/meshes/dae/R_coxa_shape.dae scale=1.0 1.0 1.0
- added link R_front_ee_link
- added link R_front_femur_link, mass 0.1; collision box size=0.10497 0.0249 0.002; visual mesh filename=package://hexapod_description/meshes/dae/R_femur_shape.dae scale=1.0 1.0 1.0
- added link R_front_foot_link, mass 0.001
- added link R_front_tibia_link, mass 0.2; collision mesh filename=package://hexapod_description/meshes/dae/R_tibia_shape.001.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 scale=1.0 1.0 1.0; visual mesh filename=package://hexapod_description/meshes/dae/R_tibia_shape.dae scale=1.0 1.0 1.0
- added link R_mid_coxa_link, mass 0.1; collision box size=0.05 0.05964 0.06371; visual mesh filename=package://hexapod_description/meshes/dae/R_coxa_shape.dae scale=1.0 1.0 1.0
- added link R_mid_ee_link
- added link R_mid_femur_link, mass 0.1; collision box size=0.10497 0.0249 0.002; visual mesh filename=package://hexapod_description/meshes/dae/R_femur_shape.dae scale=1.0 1.0 1.0
- added link R_mid_foot_link, mass 0.001
- added link R_mid_tibia_link, mass 0.2; collision mesh filename=package://hexapod_description/meshes/dae/R_tibia_shape.003.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 scale=1.0 1.0 1.0; visual mesh filename=package://hexapod_description/meshes/dae/R_tibia_shape.dae scale=1.0 1.0 1.0
- added link body_link, mass 0.2; collision box size=0.20038 0.1651 0.0538; visual mesh filename=package://hexapod_description/meshes/dae/thorax_shape.dae scale=1.0 1.0 1.0
- added link root_link
Joints:
- added joint L_back_ee_jnt: type fixed, parent L_back_foot_link, child L_back_ee_link, origin xyz=0 0 0 rpy=0 0 0
- added joint L_front_ee_jnt: type fixed, parent L_front_foot_link, child L_front_ee_link, origin xyz=0 0 0 rpy=0 0 0
- added joint L_mid_ee_jnt: type fixed, parent L_mid_foot_link, child L_mid_ee_link, origin xyz=0 0 0 rpy=0 0 0
- added joint R_back_ee_jnt: type fixed, parent R_back_foot_link, child R_back_ee_link, origin xyz=0 0 0 rpy=0 0 0
- added joint R_front_ee_jnt: type fixed, parent R_front_foot_link, child R_front_ee_link, origin xyz=0 0 0 rpy=0 0 0
- added joint R_mid_ee_jnt: type fixed, parent R_mid_foot_link, child R_mid_ee_link, origin xyz=0 0 0 rpy=0 0 0
- joint L_back_coxa_jnt: child L_back_coxa_jnt -> L_back_coxa_link; parent body_jnt -> body_link
- joint L_back_femur_jnt: child L_back_femur_jnt -> L_back_femur_link; parent L_back_coxa_jnt -> L_back_coxa_link
- joint L_back_foot_jnt: child L_back_foot_jnt -> L_back_foot_link; origin xyz=-0.13777 0.13934 -0.117 rpy=0 0 2.0944 -> xyz=0 -0.0075 -0.117 rpy=0 0 0; parent root_jnt -> L_back_tibia_link; type floating -> fixed
- joint L_back_tibia_jnt: child L_back_tibia_jnt -> L_back_tibia_link; parent L_back_femur_jnt -> L_back_femur_link
- joint L_front_coxa_jnt: child L_front_coxa_jnt -> L_front_coxa_link; parent body_jnt -> body_link
- joint L_front_femur_jnt: child L_front_femur_jnt -> L_front_femur_link; parent L_front_coxa_jnt -> L_front_coxa_link
- joint L_front_foot_jnt: child L_front_foot_jnt -> L_front_foot_link; origin xyz=0.13939 0.1384 -0.117 rpy=0 0 1.0472 -> xyz=0 -0.0075 -0.117 rpy=0 0 0; parent root_jnt -> L_front_tibia_link; type floating -> fixed
- joint L_front_tibia_jnt: child L_front_tibia_jnt -> L_front_tibia_link; parent L_front_femur_jnt -> L_front_femur_link
- joint L_mid_coxa_jnt: child L_mid_coxa_jnt -> L_mid_coxa_link; parent body_jnt -> body_link
- joint L_mid_femur_jnt: child L_mid_femur_jnt -> L_mid_femur_link; parent L_mid_coxa_jnt -> L_mid_coxa_link
- joint L_mid_foot_jnt: child L_mid_foot_jnt -> L_mid_foot_link; origin xyz=0.00094 0.17181 -0.117 rpy=0 0 1.5708 -> xyz=0 -0.0075 -0.117 rpy=0 0 0; parent root_jnt -> L_mid_tibia_link; type floating -> fixed
- joint L_mid_tibia_jnt: child L_mid_tibia_jnt -> L_mid_tibia_link; parent L_mid_femur_jnt -> L_mid_femur_link
- joint R_back_coxa_jnt: child R_back_coxa_jnt -> R_back_coxa_link; parent body_jnt -> body_link
- joint R_back_femur_jnt: child R_back_femur_jnt -> R_back_femur_link; parent R_back_coxa_jnt -> R_back_coxa_link
- joint R_back_foot_jnt: child R_back_foot_jnt -> R_back_foot_link; origin xyz=-0.13774 -0.1394 -0.117 rpy=0 0 -2.09439 -> xyz=0 -0.0075 -0.117 rpy=0 0 0; parent root_jnt -> R_back_tibia_link; type floating -> fixed
- joint R_back_tibia_jnt: child R_back_tibia_jnt -> R_back_tibia_link; parent R_back_femur_jnt -> R_back_femur_link
- joint R_front_coxa_jnt: child R_front_coxa_jnt -> R_front_coxa_link; parent body_jnt -> body_link
- joint R_front_femur_jnt: child R_front_femur_jnt -> R_front_femur_link; parent R_front_coxa_jnt -> R_front_coxa_link
- joint R_front_foot_jnt: child R_front_foot_jnt -> R_front_foot_link; origin xyz=0.13945 -0.13842 -0.117 rpy=0 0 -1.0472 -> xyz=0 -0.0075 -0.117 rpy=0 0 0; parent root_jnt -> R_front_tibia_link; type floating -> fixed
- joint R_front_tibia_jnt: child R_front_tibia_jnt -> R_front_tibia_link; parent R_front_femur_jnt -> R_front_femur_link
- joint R_mid_coxa_jnt: child R_mid_coxa_jnt -> R_mid_coxa_link; parent body_jnt -> body_link
- joint R_mid_femur_jnt: child R_mid_femur_jnt -> R_mid_femur_link; parent R_mid_coxa_jnt -> R_mid_coxa_link
- joint R_mid_foot_jnt: child R_mid_foot_jnt -> R_mid_foot_link; origin xyz=0.00099 -0.17185 -0.117 rpy=0 0 -1.5708 -> xyz=0 -0.0075 -0.117 rpy=0 0 0; parent root_jnt -> R_mid_tibia_link; type floating -> fixed
- joint R_mid_tibia_jnt: child R_mid_tibia_jnt -> R_mid_tibia_link; parent R_mid_femur_jnt -> R_mid_femur_link
- joint body_jnt: child body_jnt -> body_link; parent root_jnt -> root_link; type floating -> fixed

File: src/hexapod_description/urdf/Hexapod_gazebo.urdf (robot description, URDF)
Before this commit: robot Hexapod, 26 links, 25 joints
Links:
- removed link L_back_coxa_jnt
- removed link L_back_femur_jnt
- removed link L_back_foot_jnt
- removed link L_back_tibia_jnt
- removed link L_front_coxa_jnt
- removed link L_front_femur_jnt
- removed link L_front_foot_jnt
- removed link L_front_tibia_jnt
- removed link L_mid_coxa_jnt
- removed link L_mid_femur_jnt
- removed link L_mid_foot_jnt
- removed link L_mid_tibia_jnt
- removed link R_back_coxa_jnt
- removed link R_back_femur_jnt
- removed link R_back_foot_jnt
- removed link R_back_tibia_jnt
- removed link R_front_coxa_jnt
- removed link R_front_femur_jnt
- removed link R_front_foot_jnt
- removed link R_front_tibia_jnt
- removed link R_mid_coxa_jnt
- removed link R_mid_femur_jnt
- removed link R_mid_foot_jnt
- removed link R_mid_tibia_jnt
- removed link body_jnt
- removed link root_jnt
- added link L_back_coxa_link, mass 0.1; collision box size=0.05 0.05964 0.06371; visual mesh filename=package://hexapod_description/meshes/dae/L_coxa_shape.dae scale=1.0 1.0 1.0
- added link L_back_ee_link
- added link L_back_femur_link, mass 0.1; collision box size=0.10497 0.0249 0.002; visual mesh filename=package://hexapod_description/meshes/dae/L_femur_shape.dae scale=1.0 1.0 1.0
- added link L_back_foot_link, mass 0.001
- added link L_back_tibia_link, mass 0.2; collision mesh filename=package://hexapod_description/meshes/dae/L_tibia_shape.003.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 scale=1.0 1.0 1.0; visual mesh filename=package://hexapod_description/meshes/dae/L_tibia_shape.dae scale=1.0 1.0 1.0
- added link L_front_coxa_link, mass 0.1; collision box size=0.05 0.05964 0.06371; visual mesh filename=package://hexapod_description/meshes/dae/L_coxa_shape.dae scale=1.0 1.0 1.0
- added link L_front_ee_link
- added link L_front_femur_link, mass 0.1; collision box size=0.10497 0.0249 0.002; visual mesh filename=package://hexapod_description/meshes/dae/L_femur_shape.dae scale=1.0 1.0 1.0
- added link L_front_foot_link, mass 0.001
- added link L_front_tibia_link, mass 0.2; collision mesh filename=package://hexapod_description/meshes/dae/L_tibia_shape.001.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 scale=1.0 1.0 1.0; visual mesh filename=package://hexapod_description/meshes/dae/L_tibia_shape.dae scale=1.0 1.0 1.0
- added link L_mid_coxa_link, mass 0.1; collision box size=0.05 0.05964 0.06371; visual mesh filename=package://hexapod_description/meshes/dae/L_coxa_shape.dae scale=1.0 1.0 1.0
- added link L_mid_ee_link
- added link L_mid_femur_link, mass 0.1; collision box size=0.10497 0.0249 0.002; visual mesh filename=package://hexapod_description/meshes/dae/L_femur_shape.dae scale=1.0 1.0 1.0
- added link L_mid_foot_link, mass 0.001
- added link L_mid_tibia_link, mass 0.2; collision mesh filename=package://hexapod_description/meshes/dae/L_tibia_shape.002.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 scale=1.0 1.0 1.0; visual mesh filename=package://hexapod_description/meshes/dae/L_tibia_shape.dae scale=1.0 1.0 1.0
- added link R_back_coxa_link, mass 0.1; collision box size=0.05 0.05964 0.06371; visual mesh filename=package://hexapod_description/meshes/dae/R_coxa_shape.dae scale=1.0 1.0 1.0
- added link R_back_ee_link
- added link R_back_femur_link, mass 0.1; collision box size=0.10497 0.0249 0.002; visual mesh filename=package://hexapod_description/meshes/dae/R_femur_shape.dae scale=1.0 1.0 1.0
- added link R_back_foot_link, mass 0.001
- added link R_back_tibia_link, mass 0.2; collision mesh filename=package://hexapod_description/meshes/dae/R_tibia_shape.002.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 scale=1.0 1.0 1.0; visual mesh filename=package://hexapod_description/meshes/dae/R_tibia_shape.dae scale=1.0 1.0 1.0
- added link R_front_coxa_link, mass 0.1; collision box size=0.05 0.05964 0.06371; visual mesh filename=package://hexapod_description/meshes/dae/R_coxa_shape.dae scale=1.0 1.0 1.0
- added link R_front_ee_link
- added link R_front_femur_link, mass 0.1; collision box size=0.10497 0.0249 0.002; visual mesh filename=package://hexapod_description/meshes/dae/R_femur_shape.dae scale=1.0 1.0 1.0
- added link R_front_foot_link, mass 0.001
- added link R_front_tibia_link, mass 0.2; collision mesh filename=package://hexapod_description/meshes/dae/R_tibia_shape.001.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 scale=1.0 1.0 1.0; visual mesh filename=package://hexapod_description/meshes/dae/R_tibia_shape.dae scale=1.0 1.0 1.0
- added link R_mid_coxa_link, mass 0.1; collision box size=0.05 0.05964 0.06371; visual mesh filename=package://hexapod_description/meshes/dae/R_coxa_shape.dae scale=1.0 1.0 1.0
- added link R_mid_ee_link
- added link R_mid_femur_link, mass 0.1; collision box size=0.10497 0.0249 0.002; visual mesh filename=package://hexapod_description/meshes/dae/R_femur_shape.dae scale=1.0 1.0 1.0
- added link R_mid_foot_link, mass 0.001
- added link R_mid_tibia_link, mass 0.2; collision mesh filename=package://hexapod_description/meshes/dae/R_tibia_shape.003.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 scale=1.0 1.0 1.0; visual mesh filename=package://hexapod_description/meshes/dae/R_tibia_shape.dae scale=1.0 1.0 1.0
- added link body_link, mass 0.2; collision box size=0.20038 0.1651 0.0538; visual mesh filename=package://hexapod_description/meshes/dae/thorax_shape.dae scale=1.0 1.0 1.0
- added link root_link
Joints:
- added joint L_back_ee_jnt: type fixed, parent L_back_foot_link, child L_back_ee_link, origin xyz=0 0 0 rpy=0 0 0
- added joint L_front_ee_jnt: type fixed, parent L_front_foot_link, child L_front_ee_link, origin xyz=0 0 0 rpy=0 0 0
- added joint L_mid_ee_jnt: type fixed, parent L_mid_foot_link, child L_mid_ee_link, origin xyz=0 0 0 rpy=0 0 0
- added joint R_back_ee_jnt: type fixed, parent R_back_foot_link, child R_back_ee_link, origin xyz=0 0 0 rpy=0 0 0
- added joint R_front_ee_jnt: type fixed, parent R_front_foot_link, child R_front_ee_link, origin xyz=0 0 0 rpy=0 0 0
- added joint R_mid_ee_jnt: type fixed, parent R_mid_foot_link, child R_mid_ee_link, origin xyz=0 0 0 rpy=0 0 0
- joint L_back_coxa_jnt: child L_back_coxa_jnt -> L_back_coxa_link; parent body_jnt -> body_link
- joint L_back_femur_jnt: child L_back_femur_jnt -> L_back_femur_link; parent L_back_coxa_jnt -> L_back_coxa_link
- joint L_back_foot_jnt: child L_back_foot_jnt -> L_back_foot_link; origin xyz=-0.13777 0.13934 -0.117 rpy=0 0 2.0944 -> xyz=0 -0.0075 -0.117 rpy=0 0 0; parent root_jnt -> L_back_tibia_link; type floating -> fixed
- joint L_back_tibia_jnt: child L_back_tibia_jnt -> L_back_tibia_link; parent L_back_femur_jnt -> L_back_femur_link
- joint L_front_coxa_jnt: child L_front_coxa_jnt -> L_front_coxa_link; parent body_jnt -> body_link
- joint L_front_femur_jnt: child L_front_femur_jnt -> L_front_femur_link; parent L_front_coxa_jnt -> L_front_coxa_link
- joint L_front_foot_jnt: child L_front_foot_jnt -> L_front_foot_link; origin xyz=0.13939 0.1384 -0.117 rpy=0 0 1.0472 -> xyz=0 -0.0075 -0.117 rpy=0 0 0; parent root_jnt -> L_front_tibia_link; type floating -> fixed
- joint L_front_tibia_jnt: child L_front_tibia_jnt -> L_front_tibia_link; parent L_front_femur_jnt -> L_front_femur_link
- joint L_mid_coxa_jnt: child L_mid_coxa_jnt -> L_mid_coxa_link; parent body_jnt -> body_link
- joint L_mid_femur_jnt: child L_mid_femur_jnt -> L_mid_femur_link; parent L_mid_coxa_jnt -> L_mid_coxa_link
- joint L_mid_foot_jnt: child L_mid_foot_jnt -> L_mid_foot_link; origin xyz=0.00094 0.17181 -0.117 rpy=0 0 1.5708 -> xyz=0 -0.0075 -0.117 rpy=0 0 0; parent root_jnt -> L_mid_tibia_link; type floating -> fixed
- joint L_mid_tibia_jnt: child L_mid_tibia_jnt -> L_mid_tibia_link; parent L_mid_femur_jnt -> L_mid_femur_link
- joint R_back_coxa_jnt: child R_back_coxa_jnt -> R_back_coxa_link; parent body_jnt -> body_link
- joint R_back_femur_jnt: child R_back_femur_jnt -> R_back_femur_link; parent R_back_coxa_jnt -> R_back_coxa_link
- joint R_back_foot_jnt: child R_back_foot_jnt -> R_back_foot_link; origin xyz=-0.13774 -0.1394 -0.117 rpy=0 0 -2.09439 -> xyz=0 -0.0075 -0.117 rpy=0 0 0; parent root_jnt -> R_back_tibia_link; type floating -> fixed
- joint R_back_tibia_jnt: child R_back_tibia_jnt -> R_back_tibia_link; parent R_back_femur_jnt -> R_back_femur_link
- joint R_front_coxa_jnt: child R_front_coxa_jnt -> R_front_coxa_link; parent body_jnt -> body_link
- joint R_front_femur_jnt: child R_front_femur_jnt -> R_front_femur_link; parent R_front_coxa_jnt -> R_front_coxa_link
- joint R_front_foot_jnt: child R_front_foot_jnt -> R_front_foot_link; origin xyz=0.13945 -0.13842 -0.117 rpy=0 0 -1.0472 -> xyz=0 -0.0075 -0.117 rpy=0 0 0; parent root_jnt -> R_front_tibia_link; type floating -> fixed
- joint R_front_tibia_jnt: child R_front_tibia_jnt -> R_front_tibia_link; parent R_front_femur_jnt -> R_front_femur_link
- joint R_mid_coxa_jnt: child R_mid_coxa_jnt -> R_mid_coxa_link; parent body_jnt -> body_link
- joint R_mid_femur_jnt: child R_mid_femur_jnt -> R_mid_femur_link; parent R_mid_coxa_jnt -> R_mid_coxa_link
- joint R_mid_foot_jnt: child R_mid_foot_jnt -> R_mid_foot_link; origin xyz=0.00099 -0.17185 -0.117 rpy=0 0 -1.5708 -> xyz=0 -0.0075 -0.117 rpy=0 0 0; parent root_jnt -> R_mid_tibia_link; type floating -> fixed
- joint R_mid_tibia_jnt: child R_mid_tibia_jnt -> R_mid_tibia_link; parent R_mid_femur_jnt -> R_mid_femur_link
- joint body_jnt: child body_jnt -> body_link; parent root_jnt -> root_link; type floating -> fixed
