Commit message: update Urdf collision

File: src/hexapod_description/urdf/Hexapod.urdf (robot description, URDF)
Before this commit: robot Hexapod, 32 links, 31 joints
Links:
- link L_back_coxa_link: geometry collision mesh filename=package://hexapod_description/meshes/dae/L_coxa_shape.dae scale=1.0 1.0 1.0; visual mesh filename=package://hexapod_description/meshes/dae/L_coxa_shape.dae scale=1.0 1.0 1.0
- link L_back_femur_link: geometry collision mesh filename=package://hexapod_description/meshes/dae/L_femur_shape.dae scale=1.0 1.0 1.0; visual mesh filename=package://hexapod_description/meshes/dae/L_femur_shape.dae scale=1.0 1.0 1.0
- link L_back_tibia_link: geometry collision mesh filename=package://hexapod_description/meshes/dae/L_tibia_shape.dae scale=1.0 1.0 1.0; visual mesh filename=package://hexapod_description/meshes/dae/L_tibia_shape.dae scale=1.0 1.0 1.0
- link L_front_coxa_link: geometry collision mesh filename=package://hexapod_description/meshes/dae/L_coxa_shape.dae scale=1.0 1.0 1.0; visual mesh filename=package://hexapod_description/meshes/dae/L_coxa_shape.dae scale=1.0 1.0 1.0
- link L_front_femur_link: geometry collision mesh filename=package://hexapod_description/meshes/dae/L_femur_shape.dae scale=1.0 1.0 1.0; visual mesh filename=package://hexapod_description/meshes/dae/L_femur_shape.dae scale=1.0 1.0 1.0
- link L_front_tibia_link: geometry collision mesh filename=package://hexapod_description/meshes/dae/L_tibia_shape.dae scale=1.0 1.0 1.0; visual mesh filename=package://hexapod_description/meshes/dae/L_tibia_shape.dae scale=1.0 1.0 1.0
- link L_mid_coxa_link: geometry collision mesh filename=package://hexapod_description/meshes/dae/L_coxa_shape.dae scale=1.0 1.0 1.0; visual mesh filename=package://hexapod_description/meshes/dae/L_coxa_shape.dae scale=1.0 1.0 1.0
- link L_mid_femur_link: geometry collision mesh filename=package://hexapod_description/meshes/dae/L_femur_shape.dae scale=1.0 1.0 1.0; visual mesh filename=package://hexapod_description/meshes/dae/L_femur_shape.dae scale=1.0 1.0 1.0
- link L_mid_tibia_link: geometry collision mesh filename=package://hexapod_description/meshes/dae/L_tibia_shape.dae scale=1.0 1.0 1.0; visual mesh filename=package://hexapod_description/meshes/dae/L_tibia_shape.dae scale=1.0 1.0 1.0
- link R_back_coxa_link: geometry collision mesh filename=package://hexapod_description/meshes/dae/R_coxa_shape.dae scale=1.0 1.0 1.0; visual mesh filename=package://hexapod_description/meshes/dae/R_coxa_shape.dae scale=1.0 1.0 1.0
- link R_back_femur_link: geometry collision mesh filename=package://hexapod_description/meshes/dae/R_femur_shape.dae scale=1.0 1.0 1.0; visual mesh filename=package://hexapod_description/meshes/dae/R_femur_shape.dae scale=1.0 1.0 1.0
- link R_back_tibia_link: geometry collision mesh filename=package://hexapod_description/meshes/dae/R_tibia_shape.dae scale=1.0 1.0 1.0; visual mesh filename=package://hexapod_description/meshes/dae/R_tibia_shape.dae scale=1.0 1.0 1.0
- link R_front_coxa_link: geometry collision mesh filename=package://hexapod_description/meshes/dae/R_coxa_shape.dae scale=1.0 1.0 1.0; visual mesh filename=package://hexapod_description/meshes/dae/R_coxa_shape.dae scale=1.0 1.0 1.0
- link R_front_femur_link: geometry collision mesh filename=package://hexapod_description/meshes/dae/R_femur_shape.dae scale=1.0 1.0 1.0; visual mesh filename=package://hexapod_description/meshes/dae/R_femur_shape.dae scale=1.0 1.0 1.0
- link R_front_tibia_link: geometry collision mesh filename=package://hexapod_description/meshes/dae/R_tibia_shape.dae scale=1.0 1.0 1.0; visual mesh filename=package://hexapod_description/meshes/dae/R_tibia_shape.dae scale=1.0 1.0 1.0
- link R_mid_coxa_link: geometry collision mesh filename=package://hexapod_description/meshes/dae/R_coxa_shape.dae scale=1.0 1.0 1.0; visual mesh filename=package://hexapod_description/meshes/dae/R_coxa_shape.dae scale=1.0 1.0 1.0
- link R_mid_femur_link: geometry collision mesh filename=package://hexapod_description/meshes/dae/R_femur_shape.dae scale=1.0 1.0 1.0; visual mesh filename=package://hexapod_description/meshes/dae/R_femur_shape.dae scale=1.0 1.0 1.0
- link R_mid_tibia_link: geometry collision mesh filename=package://hexapod_description/meshes/dae/R_tibia_shape.dae scale=1.0 1.0 1.0; visual mesh filename=package://hexapod_description/meshes/dae/R_tibia_shape.dae scale=1.0 1.0 1.0
- link body_link: geometry collision mesh filename=package://hexapod_description/meshes/dae/thorax_shape.dae scale=1.0 1.0 1.0; visual mesh filename=package://hexapod_description/meshes/dae/thorax_shape.dae scale=1.0 1.0 1.0
